Commit message: inital commit

File: husky_custom_description/urdf/custom_description.urdf.xacro (robot description, xacro)
@@ -22,5 +22,5 @@
 -->
 <robot name="husky" xmlns:xacro="http://ros.org/wiki/xacro">
-  <xacro:arg name="laser_enabled" default="$(optenv HUSKY_LMS1XX_ENABLED false)" />
+  <xacro:arg name="laser_enabled" default="$(optenv HUSKY_LMS1XX_ENABLED true)" />
   <xacro:arg name="ur5_enabled" default="$(optenv HUSKY_UR5_ENABLED false)" />
   <xacro:arg name="kinect_enabled" default="false" />
@@ -28,21 +28,6 @@
   <xacro:husky_robot />
   <!-- Insert customization below, sample provided: -->
-  <link name="bowler_link">
-    <visual>
-      <geometry>
-        <mesh filename="package://husky_custom_description/meshes/red_bowler.dae" />
-      </geometry>
-    </visual>
-    <collision>
-      <origin xyz="0 0 0.07" rpy="0 0 0" />
-      <geometry>
-        <box size="0.32 0.25 0.14" rpy="0 0 0"/>
-      </geometry>
-    </collision>
-  </link>
-  <joint name="bowler_joint" type="fixed">
-    <parent link="top_plate_link" />
-    <child link="bowler_link" />
-    <origin xyz="0.1 -0.1 0" rpy="0 0 0.5" />
-  </joint>
+    <xacro:sensor_arch prefix="" parent="top_plate_link">
+        <origin xyz="0.2 0.0 0.51" rpy="0.0 0.0 0.0"/>
+    </xacro:sensor_arch>
 </robot>
